Commit message: refactor: Phase 1 single-arm setup (Robot B-centric, 7-d action, curriculum)
- Switch sim origin to Robot B (Panda) base; recompute all coords in src/config.py
- Y-split tire rack raised to Robot A base height (rail top Z = -0.30)
- Phase 1: dynamic action/obs dim (7-d / 83-d) when freeze_robot_b=True
  - Mask Panda channels in observations and action/jerk penalties
- Add approach_radius_tol curriculum (0.58 -> 0.50 m, 100k-300k steps)
  via ApproachTolCurriculumCallback in src/train.py
- Scaffold domain randomization (USE_DOMAIN_RANDOMIZATION, hub/cargo XY noise)
- HOME_POSE: UR10 tool-up, Panda ready pose (out of Robot A path)
- New scripts: train.ps1/train.bat launchers, smoke_fsm, render_phase1_goal
- Drop legacy check_* scripts; translate README.md to Korean

Co-authored-by: Cursor <cursoragent@cursor.com>

File: data/urdf/ur10_robot/ur10_robot.urdf (robot description, URDF)
Before this commit: robot ur10, 22 links, 21 joints
Links:
- link gripper_left_inner_finger: mass None -> 0.01
- link gripper_left_inner_finger_pad: mass None -> 0.01
- link gripper_left_inner_knuckle: mass None -> 0.01
- link gripper_left_outer_finger: mass None -> 0.01
- link gripper_left_outer_knuckle: mass None -> 0.01
- link gripper_right_inner_finger: mass None -> 0.01
- link gripper_right_inner_finger_pad: mass None -> 0.01
- link gripper_right_inner_knuckle: mass None -> 0.01
- link gripper_right_outer_finger: mass None -> 0.01
- link gripper_right_outer_knuckle: mass None -> 0.01
- link robot_base: mass None -> 0.01
- link robot_ee_link: mass None -> 0.01
- link robot_tool0: mass None -> 0.01

File: data/urdf/ur10_robot/ur10_robot_constr.urdf (robot description, URDF)
Before this commit: robot ur10, 22 links, 21 joints
Links:
- link gripper_left_inner_finger: mass None -> 0.01
- link gripper_left_inner_finger_pad: mass None -> 0.01
- link gripper_left_inner_knuckle: mass None -> 0.01
- link gripper_left_outer_finger: mass None -> 0.01
- link gripper_left_outer_knuckle: mass None -> 0.01
- link gripper_right_inner_finger: mass None -> 0.01
- link gripper_right_inner_finger_pad: mass None -> 0.01
- link gripper_right_inner_knuckle: mass None -> 0.01
- link gripper_right_outer_finger: mass None -> 0.01
- link gripper_right_outer_knuckle: mass None -> 0.01
- link robot_base: mass None -> 0.01
- link robot_ee_link: mass None -> 0.01
- link robot_tool0: mass None -> 0.01
