Commit message: feat(phase1): B-origin frame, reversed demount/return, pit-rim fix, drop gripper pads
- Translate whole scene -0.90 m in Y so Robot B's base lands on the world
  origin (B is now both the physical origin and the obs reference). Rigid
  translation preserves all relative geometry, reach and clearances.
- Stage 2 (demount) is now the exact reverse of the Stage-1 insertion: the
  mount EE pose translated -Y by the standoff, orientation held fixed (pure
  -Y straight pull-off, no yaw/x/z drift). Stage 3 (return) arcs
  standoff->apex->cradle, mirroring the carry arch; its redundant departure
  standoff is removed and it gets the same lift.
- Fix pit-rim collision: depth/radius had shrunk to 0.65/0.65, jamming link_2
  against the pit mouth at z=0 (~1484 N). Restore depth 0.95 / radius 0.90 so
  the buried base column is fully cleared (all stages 0 N contact).
- Remove the 3 yellow wheel-gripper pads (visual+collision) via a new
  --no-pads flag on generate_wheel_gripper_urdf.py; the tire is bonded with a
  JOINT_FIXED weld so the pads never grasped. EE/IK tip unaffected.
- Add diagnostic/verification scripts (pit, grasp orientation, yellow finder,
  hub-Y sweep, etc.).

Co-authored-by: Cursor <cursoragent@cursor.com>

File: data/urdf/fanuc_r2000ic/r2000ic210f_wheeltool.urdf (robot description, URDF)
Before this commit: robot fanuc_r2000ic210f_wheeltool, 16 links, 15 joints
Links:
- removed link wg_pad_0
- removed link wg_pad_1
- removed link wg_pad_2
Joints:
- removed joint wg_pad_0-joint
- removed joint wg_pad_1-joint
- removed joint wg_pad_2-joint

File: data/urdf/wheel_gripper/wheel_gripper.urdf (robot description, URDF)
Before this commit: robot wheel_gripper, 6 links, 5 joints
Links:
- removed link wg_pad_0
- removed link wg_pad_1
- removed link wg_pad_2
Joints:
- removed joint wg_pad_0-joint
- removed joint wg_pad_1-joint
- removed joint wg_pad_2-joint
