Commit message: fix(scene): brake proxies blocked tire seating; align mount shaping
Root-caused the curriculum stalling at frac≈0.40 (mount tol≈0.21 m) across
three reward configs: it was a geometry bug, not a reward-gradient one.

scene/URDF (the actual fix):
- brake_rotor_proxy radius 0.30 > tire bore 0.282 physically blocked the
  tire bore from sliding onto the hub — COM floored at d_A≈0.13 m, so the
  policy could only "mount" by ramming through the brakes (contact force
  124–330). Shrunk rotor to 0.22 (well inside the bore).
- Pushed brake_caliper aft (z −0.15 → −0.25) so its box (radial corner
  ≈0.35 m, inside the tread annulus) no longer intrudes into the mounting
  volume. Verified: d_A=0 now clears by ~0.02 m and a 0.04 m offset is
  collision-free in every direction, so mount_radius_tol=0.04 and the
  hub-centre mount target are reachable as-is.
- Synced generate_truck_wheel_station_urdf.py defaults to match.

reward (Stage 1 carry shaping):
- guide_A now keys on the tire→hub distance (the quantity the mount gate
  measures) instead of EE→hub; the EE-based form fought the final seating
  because the tire is fix-welded ~R below the EE.
- seat_A fine-seating kernel was tried and reverted (w_seat=0): it left
  d_A unchanged while doubling contact force and enabling a hover-and-farm
  exploit — confirming the wall was physical.

curriculum: more conservative adaptive knobs (dwell 6, advance_sr 0.85,
rollback_sr 0.50, min_episodes 60) to damp the cliff-driven oscillation.

Also bundles in-progress phase-1 WIP (tire URDF generator, teleop, robot
and scene tweaks) that was uncommitted on the working tree.

File: data/urdf/truck_assembly/truck_wheel_station.urdf (robot description, URDF)
Before this commit: robot truck_wheel_station, 14 links, 13 joints
Links:
- link brake_rotor_proxy: geometry collision cylinder length=0.022 radius=0.2178; visual cylinder length=0.022 radius=0.22
Joints:
- joint brake_caliper_joint: origin xyz=0 0.27 -0.15 rpy=0 0 0 -> xyz=0 0.27 -0.25 rpy=0 0 0
